File: HW2/ME433/schematics.brd (EAGLE design)
At the start: 50 x 50 mm, 23 parts, among them U1 PIC32MX250F128B, U2 MCP1702

Commit message: changeusb
Parts:
- USB: value USB-MB-H -> USBMINI
- moved SWITCH 1.27 mm to (17.8, 1.27)
Connections:
- removed net N$29: U1.14
- new net ID: U1.14, USB.ID
Routing:
- net ID: track 0.00 -> 34.0 mm
- net D-: track 30.0 -> 38.7 mm, vias 0 -> 2
- net D+: track 29.0 -> 23.1 mm, vias 0 -> 1
- net VBUS: track 43.3 -> 49.0 mm
- net GND: track 15.3 -> 16.6 mm

Commit message: changeposition
Parts:
- removed BUTTON1, BUTTON2: (no value), libraries:1X03
- added RESET, USER: (no value), libraries:1X03
- moved R3 9.67 mm to (11.4, 34.3), turned to 0 degrees
- moved R1 5.68 mm to (6.35, 43.2), turned to 0 degrees
- moved J1 5.39 mm to (1.27, 16.5)
- moved J2 3.42 mm to (48.9, 16.5)
- moved PICKIT 2.84 mm to (19.1, 41.9)
- moved R4 2.84 mm to (10.2, 24.1), turned to 0 degrees
- moved LED1 2.54 mm to (6.35, 47.0)
- moved R2 1.27 mm to (6.35, 39.4), turned to 180 degrees
- moved C5 1.27 mm to (29.2, 5.08)
Connections:
- net B4: now also USER.1; no longer BUTTON2.1
- net GND: now also RESET.1, USER.3; no longer BUTTON1.1, BUTTON2.3
- net MCLR: now also RESET.3; no longer BUTTON1.3
Routing:
- net B4: track 36.3 -> 49.0 mm
- net +3V3: track 132.1 -> 143.8 mm
- net A1: track 37.1 -> 42.5 mm
- net A4: track 24.7 -> 30.1 mm
- net N$1: track 4.58 -> 9.16 mm
- net B3: track 21.3 -> 25.2 mm, vias 0 -> 1
- net B2: track 21.3 -> 25.2 mm, vias 0 -> 1
- net A0: track 30.1 -> 33.9 mm, vias 0 -> 4
- net MCLR: track 27.8 -> 24.2 mm
- net B9: track 14.2 -> 17.6 mm
- net B8: track 14.2 -> 17.6 mm
- net B7: track 14.2 -> 17.6 mm
- net VBUS: track 49.0 -> 52.2 mm
- net B15: track 14.2 -> 16.7 mm
- net B14: track 14.2 -> 16.7 mm
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Other:
- board text added: "3.3V"
- board text added: "5V"
- board text added: "A0"
- board text added: "A1"
- board text added: "A4"
- board text added: "B13"
- board text added: "B14"
- board text added: "B15"
- board text added: "B2"
- board text added: "B3"
- board text added: "B4"
- board text added: "B7"
- board text added: "B8"
- board text added: "B9"
- board text added: "GND"

Commit message: gerber
Parts:
- removed RESONATOR: (no value), libraries:1X03
- added Y1: 8MHz, libraries:1X03
- C1: value 0.1uF -> 10uF
- C5: value 1uF -> 0.1uF
- moved R4 1.27 mm to (11.4, 24.1)
Connections:
- net GND: now also Y1.2; no longer RESONATOR.2
- net OSC1: now also Y1.3; no longer RESONATOR.3
- net OSC2: now also Y1.1; no longer RESONATOR.1
Routing:
- net OSC2: track 6.48 -> 5.24 mm
- net OSC1: track 6.48 -> 5.24 mm
- net GND: track 16.6 -> 15.5 mm
- net N$1: track 9.16 -> 9.92 mm
Changed lines of the file:
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@@
 <attribute name="VALUE" x="13.335" y="17.78" size="1.27" layer="27" rot="R270"/>
 </element>
-<element name="C1" library="libraries" package="C025-024X044" value="0.1uF" x="38.1" y="45.72" smashed="yes" rot="R90">
+<element name="C1" library="libraries" package="C025-024X044" value="10uF" x="38.1" y="45.72" smashed="yes" rot="R90">
 <attribute name="VALUE" x="42.418" y="45.847" size="0.8128" layer="27" ratio="10" rot="R180"/>
 </element>
@@
 <attribute name="VALUE" x="44.45" y="36.83" size="0.8128" layer="27" ratio="10"/>
 </element>
-<element name="C5" library="libraries" package="C025-024X044" value="1uF" x="29.21" y="5.08" smashed="yes" rot="R180">
+<element name="C5" library="libraries" package="C025-024X044" value="0.1uF" x="29.21" y="5.08" smashed="yes" rot="R180">
 <attribute name="VALUE" x="29.718" y="7.747" size="0.8128" layer="27" ratio="10" rot="R180"/>
 </element>
@@
 <attribute name="VALUE" x="52.07" y="15.24" size="1.27" layer="27" rot="R90"/>
 </element>
-<element name="RESONATOR" library="libraries" package="1X03" value="" x="19.05" y="20.32" smashed="yes" rot="R90">
-<attribute name="NAME" x="16.764" y="25.4762" size="0.6096" layer="25" ratio="10" rot="R270"/>
-<attribute name="VALUE" x="22.225" y="19.05" size="1.27" layer="27" rot="R90"/>
+<element name="Y1" library="libraries" package="1X03" value="8MHz" x="20.32" y="20.32" smashed="yes" rot="R90">
+<attribute name="VALUE" x="18.415" y="20.32" size="0.6096" layer="27" rot="R90"/>
 </element>
 <element name="LED1" library="led" package="LED3MM" value="" x="6.35" y="46.99" smashed="yes">
@@
 <attribute name="VALUE" x="10.668" y="32.385" size="0.6096" layer="27" ratio="10"/>
 </element>
-<element name="R4" library="resistor" package="0207/10" value="330" x="10.16" y="24.13" smashed="yes">
-<attribute name="VALUE" x="11.176" y="22.479" size="0.8128" layer="27" ratio="10" rot="R180"/>
+<element name="R4" library="resistor" package="0207/10" value="330" x="11.43" y="24.13" smashed="yes">
+<attribute name="VALUE" x="12.446" y="22.479" size="0.8128" layer="27" ratio="10" rot="R180"/>
 </element>
 <element name="U1" library="libraries" package="DIL28-3" value="PIC32MX250F128B" x="29.21" y="27.94" smashed="yes" rot="R270">
@@
 <contactref element="J1" pad="1"/>
 <contactref element="J2" pad="1"/>
-<contactref element="RESONATOR" pad="2"/>
+<contactref element="Y1" pad="2"/>
 <contactref element="C2" pad="2"/>
 <contactref element="C3" pad="2"/>
@@
 <vertex x="0" y="50.8"/>
 </polygon>
-<wire x1="19.05" y1="22.86" x2="25.4" y2="26.67" width="0.4064" layer="1"/>
+<wire x1="20.32" y1="22.86" x2="25.4" y2="26.67" width="0.4064" layer="1"/>
 <contactref element="SWITCH" pad="1.GND"/>
 <wire x1="15.78" y1="2.27" x2="16.51" y2="11.43" width="0.4064" layer="1"/>
@@
 </signal>
 <signal name="OSC1">
-<contactref element="RESONATOR" pad="3"/>
+<contactref element="Y1" pad="3"/>
 <contactref element="U1" pad="9"/>
-<wire x1="19.05" y1="25.4" x2="25.4" y2="24.13" width="0.4064" layer="16"/>
+<wire x1="20.32" y1="25.4" x2="25.4" y2="24.13" width="0.4064" layer="16"/>
 </signal>
 <signal name="OSC2">
-<contactref element="RESONATOR" pad="1"/>
+<contactref element="Y1" pad="1"/>
 <contactref element="U1" pad="10"/>
-<wire x1="19.05" y1="20.32" x2="25.4" y2="21.59" width="0.4064" layer="1"/>
+<wire x1="20.32" y1="20.32" x2="25.4" y2="21.59" width="0.4064" layer="1"/>
 </signal>
 <signal name="N$2">
@@
 <contactref element="R4" pad="2"/>
 <contactref element="LED2" pad="K"/>
-<wire x1="15.24" y1="24.13" x2="10.16" y2="16.51" width="0.4064" layer="1"/>
+<wire x1="16.51" y1="24.13" x2="10.16" y2="16.51" width="0.4064" layer="1"/>
 </signal>
 <signal name="+5V">

Commit message: Readytobecheckedbeforeorder
Parts:
- SWITCH: device libraries:SWITCH -> libraries:255SB
- moved U2 7.41 mm to (3.81, 11.4)
- moved SWITCH 5.68 mm to (12.7, 3.81), turned to 0 degrees
Connections:
- net +3V3: now also SWITCH.2
- net +5V: now also C5.1, SWITCH.1, U2.2
- net GND: no longer SWITCH.1.GND
- net VBUS: no longer C5.1, SWITCH.2.VIN, SWITCH.3.VOUT, U2.2
Routing:
- net +5V: track 0.00 -> 63.6 mm, vias 0 -> 1
- net VBUS: track 52.2 -> 8.57 mm
- net GND: track 15.5 -> 6.35 mm
- net +3V3: track 143.8 -> 146.2 mm
Other:
- board text removed: "SWITCH"
Changed lines of the file:
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@@
 <wire x1="17.78" y1="11.43" x2="17.78" y2="16.51" width="0.4064" layer="21"/>
 <wire x1="17.78" y1="16.51" x2="16.51" y2="17.78" width="0.4064" layer="21" curve="90"/>
-<text x="17.78" y="5.08" size="0.6096" layer="21">SWITCH</text>
 <wire x1="19.05" y1="49.53" x2="20.32" y2="48.26" width="0.4064" layer="21" curve="-90"/>
 <wire x1="20.32" y1="48.26" x2="19.05" y2="46.99" width="0.4064" layer="21" curve="-90"/>
@@
 <attribute name="VALUE" x="25.781" y="47.625" size="0.8128" layer="27" ratio="10"/>
 </element>
-<element name="U2" library="libraries" package="TO92" value="MCP1702" x="7.62" y="5.08" smashed="yes" rot="R90">
-<attribute name="VALUE" x="5.715" y="2.54" size="0.8128" layer="27" ratio="10" rot="R180"/>
-</element>
-<element name="SWITCH" library="libraries" package="SWITCH" value="" x="17.78" y="1.27" smashed="yes" rot="R90"/>
+<element name="U2" library="libraries" package="TO92" value="MCP1702" x="3.81" y="11.43" smashed="yes" rot="R90">
+<attribute name="VALUE" x="5.842" y="11.557" size="0.8128" layer="27" ratio="10" rot="R270"/>
+</element>
 <element name="USB" library="libraries" package="USB-MB-H" value="USBMINI" x="44.45" y="7.62" smashed="yes" rot="R180">
 <attribute name="NAME" x="39.6" y="12.446" size="0.8128" layer="25"/>
+</element>
+<element name="SWITCH" library="libraries" package="255SB" value="" x="12.7" y="3.81" smashed="yes">
+<attribute name="NAME" x="7.112" y="7.366" size="0.8128" layer="25" ratio="10"/>
+<attribute name="VALUE" x="12.7" y="7.366" size="1.27" layer="27" ratio="10"/>
 </element>
 </elements>
@@
 <wire x1="44.45" y1="44.45" x2="44.45" y2="39.37" width="0.4064" layer="1"/>
 <wire x1="38.1" y1="40.64" x2="38.1" y2="44.45" width="0.4064" layer="1"/>
-<wire x1="7.62" y1="6.35" x2="20.32" y2="10.16" width="0.4064" layer="16"/>
 <wire x1="25.4" y1="13.97" x2="27.94" y2="13.97" width="0.4064" layer="1"/>
 <wire x1="27.94" y1="13.97" x2="30.48" y2="16.51" width="0.4064" layer="1"/>
@@
 <wire x1="7.62" y1="36.83" x2="16.51" y2="36.83" width="0.4064" layer="1"/>
 <wire x1="16.51" y1="36.83" x2="19.05" y2="39.37" width="0.4064" layer="1"/>
-<wire x1="1.27" y1="19.05" x2="2.54" y2="19.05" width="0.4064" layer="1"/>
-<wire x1="2.54" y1="19.05" x2="3.81" y2="17.78" width="0.4064" layer="1"/>
-<wire x1="3.81" y1="17.78" x2="3.81" y2="10.16" width="0.4064" layer="1"/>
-<wire x1="3.81" y1="10.16" x2="7.62" y2="6.35" width="0.4064" layer="1"/>
+<contactref element="SWITCH" pad="2"/>
+<wire x1="3.81" y1="12.7" x2="3.81" y2="17.78" width="0.4064" layer="16"/>
+<wire x1="3.81" y1="17.78" x2="2.54" y2="19.05" width="0.4064" layer="16"/>
+<wire x1="2.54" y1="19.05" x2="1.27" y2="19.05" width="0.4064" layer="16"/>
+<wire x1="3.81" y1="12.7" x2="5.08" y2="12.7" width="0.4064" layer="16"/>
+<wire x1="5.08" y1="12.7" x2="12.7" y2="5.08" width="0.4064" layer="16" curve="-90"/>
+<wire x1="12.7" y1="5.08" x2="12.7" y2="3.81" width="0.4064" layer="16"/>
+<wire x1="20.32" y1="10.16" x2="19.05" y2="10.16" width="0.4064" layer="1"/>
+<wire x1="19.05" y1="10.16" x2="12.7" y2="3.81" width="0.4064" layer="1"/>
 </signal>
 <signal name="GND">
@@
 </polygon>
 <wire x1="20.32" y1="22.86" x2="25.4" y2="26.67" width="0.4064" layer="1"/>
-<contactref element="SWITCH" pad="1.GND"/>
-<wire x1="15.78" y1="2.27" x2="16.51" y2="11.43" width="0.4064" layer="1"/>
 <contactref element="USB" pad="GND"/>
+<wire x1="3.81" y1="10.16" x2="1.27" y2="16.51" width="0" layer="19" extent="1-1"/>
 </signal>
 <signal name="A0">
@@
 <signal name="VBUS">
 <contactref element="U1" pad="15"/>
-<contactref element="C5" pad="1"/>
-<contactref element="SWITCH" pad="2.VIN"/>
-<contactref element="U2" pad="2"/>
-<contactref element="SWITCH" pad="3.VOUT"/>
-<wire x1="17.78" y1="2.27" x2="19.78" y2="2.27" width="0.4064" layer="16"/>
-<wire x1="5.715" y1="5.08" x2="16.51" y2="5.08" width="0.4064" layer="16"/>
-<wire x1="16.51" y1="5.08" x2="17.78" y2="2.27" width="0.4064" layer="16"/>
-<wire x1="19.78" y1="2.27" x2="20.05" y2="3.54" width="0.4064" layer="16"/>
 <contactref element="USB" pad="VBUS"/>
-<wire x1="30.48" y1="5.08" x2="30.48" y2="8.89" width="0.4064" layer="16"/>
-<wire x1="30.48" y1="8.89" x2="33.02" y2="11.43" width="0.4064" layer="16"/>
-<wire x1="39.35" y1="6.02" x2="33.35" y2="6.02" width="0.4064" layer="16"/>
-<wire x1="33.35" y1="6.02" x2="33.02" y2="6.35" width="0.4064" layer="16"/>
-<wire x1="33.02" y1="6.35" x2="33.02" y2="11.43" width="0.4064" layer="16"/>
-<wire x1="30.48" y1="5.08" x2="30.48" y2="3.81" width="0.4064" layer="16"/>
-<wire x1="30.48" y1="3.81" x2="29.21" y2="2.54" width="0.4064" layer="16"/>
-<wire x1="29.21" y1="2.54" x2="24.13" y2="2.54" width="0.4064" layer="16"/>
-<wire x1="24.13" y1="2.54" x2="24.13" y2="3.81" width="0.4064" layer="16"/>
-<wire x1="24.13" y1="3.81" x2="22.86" y2="5.08" width="0.4064" layer="16"/>
-<wire x1="22.86" y1="5.08" x2="21.59" y2="5.08" width="0.4064" layer="16"/>
-<wire x1="21.59" y1="5.08" x2="20.32" y2="3.81" width="0.4064" layer="16"/>
-<wire x1="20.32" y1="3.81" x2="20.32" y2="2.81" width="0.4064" layer="16"/>
-<wire x1="20.32" y1="2.81" x2="19.78" y2="2.27" width="0.4064" layer="16"/>
+<wire x1="39.35" y1="6.02" x2="38.43" y2="6.02" width="0.4064" layer="16"/>
+<wire x1="38.43" y1="6.02" x2="33.02" y2="11.43" width="0.4064" layer="16"/>
 </signal>
 <signal name="MCLR">
@@
 <signal name="+5V">
 <contactref element="J2" pad="2"/>
+<contactref element="C5" pad="1"/>
+<contactref element="U2" pad="2"/>
+<contactref element="SWITCH" pad="1"/>
+<wire x1="1.905" y1="11.43" x2="1.905" y2="6.985" width="0.4064" layer="16"/>
+<wire x1="1.905" y1="6.985" x2="7.62" y2="1.27" width="0.4064" layer="16" curve="90"/>
+<wire x1="7.62" y1="1.27" x2="8.16" y2="1.27" width="0.4064" layer="16"/>
+<wire x1="8.16" y1="1.27" x2="10.7" y2="3.81" width="0.4064" layer="16" curve="90"/>
+<wire x1="30.48" y1="5.08" x2="26.67" y2="1.27" width="0.4064" layer="16" curve="-90"/>
+<wire x1="26.67" y1="1.27" x2="12.7" y2="1.27" width="0.4064" layer="16"/>
+<wire x1="12.7" y1="1.27" x2="10.7" y2="3.27" width="0.4064" layer="16" curve="-90"/>
+<wire x1="10.7" y1="3.27" x2="10.7" y2="3.81" width="0.4064" layer="16"/>
+<wire x1="30.48" y1="5.08" x2="31.75" y2="5.08" width="0.4064" layer="16"/>
+<wire x1="31.75" y1="5.08" x2="34.29" y2="7.62" width="0.4064" layer="16"/>
+<via x="34.29" y="7.62" extent="1-16" drill="0.6" shape="square"/>
+<wire x1="34.29" y1="7.62" x2="43.18" y2="16.51" width="0.4064" layer="1"/>
+<wire x1="43.18" y1="16.51" x2="46.355" y2="16.51" width="0.4064" layer="1"/>
+<wire x1="46.355" y1="16.51" x2="48.895" y2="19.05" width="0.4064" layer="1"/>
 </signal>
 <signal name="ID">
