File: HW2/ME433/schematics.sch (EAGLE design)
At the start: 23 parts, among them U1 PIC32MX250F128B, U2 MCP1702

Commit message: changeusb
Parts:
- USB: value USB-MB-H -> USBMINI; device libraries:USB-MB-H -> libraries:USBMINI
Connections:
- removed net N$29: U1.14.USBID/RB5
- new net ID: U1.14.USBID/RB5, USB.2.ID
- net D+: now also USB.3.D+; no longer USB.D+
- net D-: now also USB.4.D-; no longer USB.D-
- net GND: now also USB.1.GND; no longer USB.GND
- net VBUS: now also USB.5.VBUS; no longer USB.VBUS
Other:
- moved on the sheet: SWITCH
Changed lines of the file:
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@@
 <part name="C2" library="libraries" deviceset="C-US" device="025-024X044" value="0.1uF"/>
 <part name="GND2" library="libraries" deviceset="GND" device=""/>
-<part name="USB" library="libraries" deviceset="USB" device="-MB-H"/>
 <part name="C3" library="libraries" deviceset="C-US" device="025-024X044" value="10uF"/>
 <part name="GND3" library="libraries" deviceset="GND" device=""/>
@@
 <part name="P+1" library="libraries" deviceset="+5V" device=""/>
 <part name="SWITCH" library="libraries" deviceset="SWITCH" device=""/>
+<part name="USB" library="libraries" deviceset="USBMINI" device=""/>
 </parts>
 <sheets>
@@
 <instance part="C2" gate="G$1" x="38.1" y="-15.24"/>
 <instance part="GND2" gate="1" x="38.1" y="-27.94"/>
-<instance part="USB" gate="G$1" x="78.74" y="-30.48"/>
 <instance part="C3" gate="G$1" x="109.22" y="15.24" rot="R90"/>
 <instance part="GND3" gate="1" x="119.38" y="15.24" rot="R90"/>
@@
 <instance part="P+1" gate="1" x="132.08" y="-71.12" rot="R270"/>
 <instance part="SWITCH" gate="G$1" x="66.04" y="129.54"/>
+<instance part="USB" gate="G$1" x="167.64" y="-7.62"/>
 </instances>
 <busses>
@@
 </segment>
 <segment>
-<pinref part="USB" gate="G$1" pin="GND"/>
-<wire x1="76.2" y1="-30.48" x2="66.04" y2="-30.48" width="0.1524" layer="91"/>
-<label x="66.04" y="-30.48" size="1.778" layer="95"/>
-</segment>
-<segment>
 <pinref part="C3" gate="G$1" pin="2"/>
 <wire x1="114.3" y1="15.24" x2="116.84" y2="15.24" width="0.1524" layer="91"/>
@@
 <label x="48.26" y="127" size="1.778" layer="95"/>
 </segment>
+<segment>
+<pinref part="USB" gate="G$1" pin="1.GND"/>
+<wire x1="147.32" y1="2.54" x2="134.62" y2="2.54" width="0.1524" layer="91"/>
+<label x="137.16" y="2.54" size="1.778" layer="95"/>
+</segment>
 </net>
 <net name="A0" class="0">
@@
 </segment>
 <segment>
-<pinref part="USB" gate="G$1" pin="D+"/>
-<wire x1="76.2" y1="-22.86" x2="66.04" y2="-22.86" width="0.1524" layer="91"/>
-<label x="66.04" y="-22.86" size="1.778" layer="95"/>
+<pinref part="USB" gate="G$1" pin="3.D+"/>
+<wire x1="147.32" y1="-7.62" x2="134.62" y2="-7.62" width="0.1524" layer="91"/>
+<label x="137.16" y="-7.62" size="1.778" layer="95"/>
 </segment>
 </net>
@@
 </segment>
 <segment>
-<pinref part="USB" gate="G$1" pin="D-"/>
-<wire x1="76.2" y1="-25.4" x2="66.04" y2="-25.4" width="0.1524" layer="91"/>
-<label x="66.04" y="-25.4" size="1.778" layer="95"/>
-<label x="66.04" y="-25.4" size="1.778" layer="95"/>
+<pinref part="USB" gate="G$1" pin="4.D-"/>
+<wire x1="147.32" y1="-12.7" x2="134.62" y2="-12.7" width="0.1524" layer="91"/>
+<label x="137.16" y="-12.7" size="1.778" layer="95"/>
 </segment>
 </net>
@@
 <wire x1="99.06" y1="-10.16" x2="104.14" y2="-10.16" width="0.1524" layer="91"/>
 <label x="101.6" y="-10.16" size="1.778" layer="95"/>
-</segment>
-<segment>
-<pinref part="USB" gate="G$1" pin="VBUS"/>
-<wire x1="76.2" y1="-27.94" x2="66.04" y2="-27.94" width="0.1524" layer="91"/>
-<label x="66.04" y="-27.94" size="1.778" layer="95"/>
 </segment>
 <segment>
@@
 <label x="48.26" y="124.46" size="1.778" layer="95"/>
 </segment>
-</net>
-<net name="N$29" class="0">
-<segment>
-<pinref part="U1" gate="G$1" pin="14.USBID/RB5"/>
-<wire x1="48.26" y1="-10.16" x2="43.18" y2="-10.16" width="0.1524" layer="91"/>
+<segment>
+<pinref part="USB" gate="G$1" pin="5.VBUS"/>
+<wire x1="147.32" y1="-17.78" x2="134.62" y2="-17.78" width="0.1524" layer="91"/>
+<label x="137.16" y="-17.78" size="1.778" layer="95"/>
 </segment>
 </net>
@@
 </segment>
 </net>
+<net name="ID" class="0">
+<segment>
+<pinref part="USB" gate="G$1" pin="2.ID"/>
+<wire x1="147.32" y1="-2.54" x2="134.62" y2="-2.54" width="0.1524" layer="91"/>
+<label x="137.16" y="-2.54" size="1.778" layer="95"/>
+</segment>
+<segment>
+<pinref part="U1" gate="G$1" pin="14.USBID/RB5"/>
+<wire x1="48.26" y1="-10.16" x2="43.18" y2="-10.16" width="0.1524" layer="91"/>
+<label x="43.18" y="-10.16" size="1.778" layer="95"/>
+</segment>
+</net>

Commit message: changeposition
Parts:
- renumbered BUTTON1 to RESET, BUTTON2 to USER
Other:
- moved on the sheet: R1
Changed lines of the file:
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@@
 <part name="C1" library="libraries" deviceset="C-US" device="025-024X044" value="0.1uF"/>
 <part name="C4" library="libraries" deviceset="C-US" device="025-024X044" value="0.1uF"/>
-<part name="BUTTON1" library="libraries" deviceset="M03" device="PTH"/>
+<part name="RESET" library="libraries" deviceset="M03" device="PTH"/>
 <part name="R2" library="libraries" deviceset="R-US_" device="0207/10" value="10k"/>
 <part name="R3" library="libraries" deviceset="R-US_" device="0207/10" value="10k"/>
-<part name="BUTTON2" library="libraries" deviceset="M03" device="PTH"/>
+<part name="USER" library="libraries" deviceset="M03" device="PTH"/>
 <part name="LED2" library="led" deviceset="LED" device="3MM"/>
 <part name="R4" library="resistor" deviceset="R-US_" device="0207/10" value="330"/>
@@
 <instance part="C1" gate="G$1" x="127" y="30.48" rot="R90"/>
 <instance part="C4" gate="G$1" x="119.38" y="55.88" rot="R90"/>
-<instance part="BUTTON1" gate="J$1" x="15.24" y="53.34"/>
+<instance part="RESET" gate="J$1" x="15.24" y="53.34"/>
 <instance part="R2" gate="G$1" x="33.02" y="66.04" rot="R90"/>
 <instance part="R3" gate="G$1" x="12.7" y="5.08"/>
-<instance part="BUTTON2" gate="J$1" x="12.7" y="22.86"/>
+<instance part="USER" gate="J$1" x="12.7" y="22.86"/>
 <instance part="LED2" gate="G$1" x="-7.62" y="-17.78"/>
 <instance part="R4" gate="G$1" x="-7.62" y="-33.02" rot="R90"/>
@@
 <instance part="GND7" gate="1" x="129.54" y="106.68" rot="R90"/>
 <instance part="LED1" gate="G$1" x="20.32" y="-38.1"/>
-<instance part="R1" gate="G$1" x="20.32" y="-53.34" rot="R90"/>
+<instance part="R1" gate="G$1" x="20.32" y="-50.8" rot="R90"/>
 <instance part="GND8" gate="1" x="20.32" y="-68.58"/>
 <instance part="+3V1" gate="G$1" x="20.32" y="-25.4"/>
@@
 </segment>
 <segment>
-<pinref part="BUTTON1" gate="J$1" pin="1"/>
+<pinref part="RESET" gate="J$1" pin="1"/>
 <wire x1="22.86" y1="50.8" x2="27.94" y2="50.8" width="0.1524" layer="91"/>
 <label x="25.4" y="50.8" size="1.778" layer="95"/>
@@
 </segment>
 <segment>
-<pinref part="BUTTON2" gate="J$1" pin="3"/>
+<pinref part="USER" gate="J$1" pin="3"/>
 <wire x1="20.32" y1="25.4" x2="27.94" y2="27.94" width="0.1524" layer="91"/>
 <wire x1="27.94" y1="27.94" x2="27.94" y2="33.02" width="0.1524" layer="91"/>
@@
 <pinref part="GND8" gate="1" pin="GND"/>
 <pinref part="R1" gate="G$1" pin="1"/>
-<wire x1="20.32" y1="-66.04" x2="20.32" y2="-58.42" width="0.1524" layer="91"/>
+<wire x1="20.32" y1="-66.04" x2="20.32" y2="-55.88" width="0.1524" layer="91"/>
 </segment>
 <segment>
@@
 <label x="43.18" y="5.08" size="1.778" layer="95"/>
 <wire x1="17.78" y1="5.08" x2="20.32" y2="5.08" width="0.1524" layer="91"/>
-<pinref part="BUTTON2" gate="J$1" pin="1"/>
+<pinref part="USER" gate="J$1" pin="1"/>
 <wire x1="20.32" y1="5.08" x2="48.26" y2="5.08" width="0.1524" layer="91"/>
 <wire x1="20.32" y1="20.32" x2="20.32" y2="5.08" width="0.1524" layer="91"/>
@@
 <junction x="45.72" y="55.88"/>
 <label x="45.72" y="60.96" size="1.778" layer="95"/>
-<pinref part="BUTTON1" gate="J$1" pin="3"/>
+<pinref part="RESET" gate="J$1" pin="3"/>
 <wire x1="33.02" y1="55.88" x2="33.02" y2="60.96" width="0.1524" layer="91"/>
 <junction x="33.02" y="55.88"/>
@@
 <pinref part="R1" gate="G$1" pin="2"/>
 <pinref part="LED1" gate="G$1" pin="C"/>
-<wire x1="20.32" y1="-48.26" x2="20.32" y2="-43.18" width="0.1524" layer="91"/>
-</segment>
-</net>
+<wire x1="20.32" y1="-45.72" x2="20.32" y2="-43.18" width="0.1524" layer="91"/>
+</segment>
+</net>

Commit message: gerber
Parts:
- C1: value 0.1uF -> 10uF
- C5: value 1uF -> 0.1uF
- Y1: value (none) -> 8MHz
- renumbered RESONATOR to Y1
Changed lines of the file:
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@@
 <part name="PICKIT" library="libraries" deviceset="M05" device="PTH"/>
 <part name="+3V2" library="libraries" deviceset="+3V3" device=""/>
-<part name="RESONATOR" library="libraries" deviceset="M03" device="PTH"/>
+<part name="Y1" library="libraries" deviceset="M03" device="PTH" value="8MHz"/>
 <part name="+3V3" library="libraries" deviceset="+3V3" device=""/>
 <part name="C2" library="libraries" deviceset="C-US" device="025-024X044" value="0.1uF"/>
@@
 <part name="GND3" library="libraries" deviceset="GND" device=""/>
 <part name="GND4" library="libraries" deviceset="GND" device=""/>
-<part name="C1" library="libraries" deviceset="C-US" device="025-024X044" value="0.1uF"/>
+<part name="C1" library="libraries" deviceset="C-US" device="025-024X044" value="10uF"/>
 <part name="C4" library="libraries" deviceset="C-US" device="025-024X044" value="0.1uF"/>
 <part name="RESET" library="libraries" deviceset="M03" device="PTH"/>
@@
 <part name="GND5" library="supply1" deviceset="GND" device=""/>
 <part name="GND1" library="supply1" deviceset="GND" device=""/>
-<part name="C5" library="libraries" deviceset="C-US" device="025-024X044" value="1uF"/>
+<part name="C5" library="libraries" deviceset="C-US" device="025-024X044" value="0.1uF"/>
 <part name="C6" library="libraries" deviceset="C-US" device="025-024X044" value="10uF"/>
 <part name="C7" library="libraries" deviceset="C-US" device="025-024X044" value="0.1uF"/>
@@
 <instance part="PICKIT" gate="G$1" x="71.12" y="-55.88"/>
 <instance part="+3V2" gate="G$1" x="-2.54" y="48.26"/>
-<instance part="RESONATOR" gate="J$1" x="-20.32" y="15.24"/>
+<instance part="Y1" gate="J$1" x="-20.32" y="15.24"/>
 <instance part="+3V3" gate="G$1" x="33.02" y="-5.08" rot="R90"/>
 <instance part="C2" gate="G$1" x="38.1" y="-15.24"/>
@@
 </segment>
 <segment>
-<pinref part="RESONATOR" gate="J$1" pin="2"/>
+<pinref part="Y1" gate="J$1" pin="2"/>
 <wire x1="-12.7" y1="15.24" x2="-10.16" y2="15.24" width="0.1524" layer="91"/>
 <label x="-10.16" y="15.24" size="1.778" layer="95"/>
@@
 <net name="OSC1" class="0">
 <segment>
-<pinref part="RESONATOR" gate="J$1" pin="3"/>
+<pinref part="Y1" gate="J$1" pin="3"/>
 <wire x1="-12.7" y1="17.78" x2="-7.62" y2="17.78" width="0.1524" layer="91"/>
 <label x="-10.16" y="17.78" size="1.778" layer="95"/>
@@
 <net name="OSC2" class="0">
 <segment>
-<pinref part="RESONATOR" gate="J$1" pin="1"/>
+<pinref part="Y1" gate="J$1" pin="1"/>
 <wire x1="-12.7" y1="12.7" x2="-7.62" y2="12.7" width="0.1524" layer="91"/>
 <label x="-10.16" y="12.7" size="1.778" layer="95"/>

Commit message: Readytobecheckedbeforeorder
Parts:
- SWITCH: device libraries:SWITCH -> libraries:255SB
Connections:
- net +3V3: now also SWITCH.P
- net +5V: now also C5.1, SWITCH.O, U2.2.VIN
- net GND: no longer SWITCH.1.GND
- net VBUS: no longer C5.1, SWITCH.2.VIN, SWITCH.3.VOUT, U2.2.VIN
Changed lines of the file:
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@@
 <part name="GND11" library="libraries" deviceset="GND" device=""/>
 <part name="P+1" library="libraries" deviceset="+5V" device=""/>
-<part name="SWITCH" library="libraries" deviceset="SWITCH" device=""/>
 <part name="USB" library="libraries" deviceset="USBMINI" device=""/>
+<part name="SWITCH" library="libraries" deviceset="255SB" device=""/>
+<part name="P+2" library="libraries" deviceset="+5V" device=""/>
 </parts>
 <sheets>
@@
 <instance part="GND11" gate="1" x="27.94" y="35.56" rot="R180"/>
 <instance part="P+1" gate="1" x="132.08" y="-71.12" rot="R270"/>
-<instance part="SWITCH" gate="G$1" x="66.04" y="129.54"/>
 <instance part="USB" gate="G$1" x="167.64" y="-7.62"/>
+<instance part="SWITCH" gate="1" x="35.56" y="127" rot="R90"/>
+<instance part="P+2" gate="1" x="22.86" y="106.68" rot="R90"/>
 </instances>
 <busses>
@@
 <junction x="86.36" y="106.68"/>
 <label x="86.36" y="96.52" size="1.778" layer="95"/>
+<wire x1="86.36" y1="129.54" x2="86.36" y2="106.68" width="0.1524" layer="91"/>
+<junction x="86.36" y="106.68"/>
+<pinref part="SWITCH" gate="1" pin="P"/>
+<wire x1="40.64" y1="129.54" x2="86.36" y2="129.54" width="0.1524" layer="91"/>
 </segment>
 </net>
@@
 </segment>
 <segment>
-<pinref part="SWITCH" gate="G$1" pin="1.GND"/>
-<wire x1="60.96" y1="127" x2="48.26" y2="127" width="0.1524" layer="91"/>
-<label x="48.26" y="127" size="1.778" layer="95"/>
-</segment>
-<segment>
 <pinref part="USB" gate="G$1" pin="1.GND"/>
 <wire x1="147.32" y1="2.54" x2="134.62" y2="2.54" width="0.1524" layer="91"/>
@@
 <wire x1="99.06" y1="-10.16" x2="104.14" y2="-10.16" width="0.1524" layer="91"/>
 <label x="101.6" y="-10.16" size="1.778" layer="95"/>
-</segment>
-<segment>
-<pinref part="C5" gate="G$1" pin="1"/>
-<wire x1="35.56" y1="106.68" x2="25.4" y2="106.68" width="0.1524" layer="91"/>
-<wire x1="35.56" y1="96.52" x2="35.56" y2="106.68" width="0.1524" layer="91"/>
-<label x="25.4" y="106.68" size="1.778" layer="95"/>
-<pinref part="U2" gate="G$1" pin="2.VIN"/>
-<wire x1="45.72" y1="106.68" x2="40.64" y2="106.68" width="0.1524" layer="91"/>
-<junction x="35.56" y="106.68"/>
-<pinref part="SWITCH" gate="G$1" pin="3.VOUT"/>
-<wire x1="40.64" y1="106.68" x2="35.56" y2="106.68" width="0.1524" layer="91"/>
-<wire x1="60.96" y1="121.92" x2="40.64" y2="121.92" width="0.1524" layer="91"/>
-<wire x1="40.64" y1="121.92" x2="40.64" y2="106.68" width="0.1524" layer="91"/>
-<junction x="40.64" y="106.68"/>
-</segment>
-<segment>
-<pinref part="SWITCH" gate="G$1" pin="2.VIN"/>
-<wire x1="60.96" y1="124.46" x2="48.26" y2="124.46" width="0.1524" layer="91"/>
-<label x="48.26" y="124.46" size="1.778" layer="95"/>
 </segment>
 <segment>
@@
 <pinref part="P+1" gate="1" pin="+5V"/>
 </segment>
-</net>
+<segment>
+<pinref part="C5" gate="G$1" pin="1"/>
+<wire x1="35.56" y1="106.68" x2="25.4" y2="106.68" width="0.1524" layer="91"/>
+<wire x1="35.56" y1="96.52" x2="35.56" y2="106.68" width="0.1524" layer="91"/>
+<pinref part="U2" gate="G$1" pin="2.VIN"/>
+<wire x1="45.72" y1="106.68" x2="38.1" y2="106.68" width="0.1524" layer="91"/>
+<junction x="35.56" y="106.68"/>
+<wire x1="38.1" y1="106.68" x2="35.56" y2="106.68" width="0.1524" layer="91"/>
+<pinref part="SWITCH" gate="1" pin="O"/>
+<wire x1="30.48" y1="127" x2="30.48" y2="109.22" width="0.1524" layer="91"/>
+<wire x1="30.48" y1="109.22" x2="38.1" y2="109.22" width="0.1524" layer="91"/>
+<wire x1="38.1" y1="109.22" x2="38.1" y2="106.68" width="0.1524" layer="91"/>
+<junction x="38.1" y="106.68"/>
+<pinref part="P+2" gate="1" pin="+5V"/>
+</segment>
+</net>
